File: Hardware/Dev Board/Rev 1.0/Dev Board.kicad_pcb (KiCad board)
At the start: 2 copper layers, 100 x 100 mm, 46 parts, among them J1 VBAT, J2 SPI, J3 PANEL, J4 6502 Card Connector, J5 6502 Bus, J6 USB Host, J7 USB HOST, J8 RJ45_LED, J9 ETHERNET, SW1 Run/Stop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

Commit message: Uppercase DEV
Parts:
- G***: footprint 6502 Logos:6502 Dev Board Logo 4mm -> 6502 Logos:6502 DEV Board Logo 4mm
Changed lines of the file:
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@@
 	(paper "USLetter")
 	(title_block
-		(title "6502 Dev Board")
+		(title "6502 DEV Board")
 		(date "2025-09-26")
 		(rev "1.0")
@@
 		(property ki_fp_filters "MountingHole*")
 		(sheetname "/")
-		(sheetfile "Dev Board.kicad_sch")
+		(sheetfile "DEV Board.kicad_sch")
 		(attr board_only exclude_from_pos_files exclude_from_bom)
 		(duplicate_pad_numbers_are_jumpers no)
@@
 		(property ki_fp_filters "MountingHole*")
 		(sheetname "/")
-		(sheetfile "Dev Board.kicad_sch")
+		(sheetfile "DEV Board.kicad_sch")
 		(attr board_only exclude_from_pos_files exclude_from_bom)
 		(duplicate_pad_numbers_are_jumpers no)
@@
 		(property ki_fp_filters "MountingHole*")
 		(sheetname "/")
-		(sheetfile "Dev Board.kicad_sch")
+		(sheetfile "DEV Board.kicad_sch")
 		(attr board_only exclude_from_pos_files exclude_from_bom)
 		(duplicate_pad_numbers_are_jumpers no)
@@
 		(property ki_fp_filters "MountingHole*")
 		(sheetname "/")
-		(sheetfile "Dev Board.kicad_sch")
+		(sheetfile "DEV Board.kicad_sch")
 		(attr board_only exclude_from_pos_files exclude_from_bom)
 		(duplicate_pad_numbers_are_jumpers no)
@@
 		(property ki_fp_filters "Connector*:*_1x??_*")
 		(sheetname "/")
-		(sheetfile "Dev Board.kicad_sch")
+		(sheetfile "DEV Board.kicad_sch")
 		(units
 			(unit
@@
 		(property ki_fp_filters "R_*")
 		(sheetname "/")
-		(sheetfile "Dev Board.kicad_sch")
+		(sheetfile "DEV Board.kicad_sch")
 		(units
 			(unit
@@
 		(property ki_fp_filters "Connector*:*_2x??_*")
 		(sheetname "/")
-		(sheetfile "Dev Board.kicad_sch")
+		(sheetfile "DEV Board.kicad_sch")
 		(attr through_hole)
 		(duplicate_pad_numbers_are_jumpers no)
@@
 		(embedded_fonts no)
 	)
-	(footprint "6502 Logos:6502 Dev Board Logo 4mm"
+	(footprint "6502 Logos:6502 DEV Board Logo 4mm"
 		(layer "F.Cu")
 		(at 166.719057 56.139968 180)
@@
 		)
 		(sheetname "/")
-		(sheetfile "Dev Board.kicad_sch")
+		(sheetfile "DEV Board.kicad_sch")
 		(attr through_hole)
 		(duplicate_pad_numbers_are_jumpers no)
@@
 		(property ki_fp_filters "R_*")
 		(sheetname "/")
-		(sheetfile "Dev Board.kicad_sch")
+		(sheetfile "DEV Board.kicad_sch")
 		(units
 			(unit
@@
 		(property ki_fp_filters "Connector*:*_2x??_*")
 		(sheetname "/")
-		(sheetfile "Dev Board.kicad_sch")
+		(sheetfile "DEV Board.kicad_sch")
 		(units
 			(unit
@@
 		)
 		(sheetname "/")
-		(sheetfile "Dev Board.kicad_sch")
+		(sheetfile "DEV Board.kicad_sch")
 		(units
 			(unit
@@
 		(property ki_fp_filters "R_*")
 		(sheetname "/")
-		(sheetfile "Dev Board.kicad_sch")
+		(sheetfile "DEV Board.kicad_sch")
 		(units
 			(unit
@@
 		(property ki_fp_filters "C_*")
 		(sheetname "/")
-		(sheetfile "Dev Board.kicad_sch")
+		(sheetfile "DEV Board.kicad_sch")
 		(units
 			(unit
@@
 		)
 		(sheetname "/")
-		(sheetfile "Dev Board.kicad_sch")
+		(sheetfile "DEV Board.kicad_sch")
 		(attr through_hole)
 		(duplicate_pad_numbers_are_jumpers no)
@@
 		)
 		(sheetname "/")
-		(sheetfile "Dev Board.kicad_sch")
+		(sheetfile "DEV Board.kicad_sch")
 		(attr through_hole)
 		(duplicate_pad_numbers_are_jumpers no)
@@
 		)
 		(sheetname "/")
-		(sheetfile "Dev Board.kicad_sch")
+		(sheetfile "DEV Board.kicad_sch")
 		(attr through_hole)
 		(duplicate_pad_numbers_are_jumpers no)
@@
 		(property ki_fp_filters "R_*")
 		(sheetname "/")
-		(sheetfile "Dev Board.kicad_sch")
+		(sheetfile "DEV Board.kicad_sch")
 		(units
 			(unit
@@
 		(property ki_fp_filters "Connector*:*_2x??_*")
 		(sheetname "/")
-		(sheetfile "Dev Board.kicad_sch")
+		(sheetfile "DEV Board.kicad_sch")
 		(units
 			(unit
@@
 		(property ki_fp_filters "R_*")
 		(sheetname "/")
-		(sheetfile "Dev Board.kicad_sch")
+		(sheetfile "DEV Board.kicad_sch")
 		(units
 			(unit
@@
 		(property ki_fp_filters "C_*")
 		(sheetname "/")
-		(sheetfile "Dev Board.kicad_sch")
+		(sheetfile "DEV Board.kicad_sch")
 		(units
 			(unit
@@
 		)
 		(sheetname "/")
-		(sheetfile "Dev Board.kicad_sch")
+		(sheetfile "DEV Board.kicad_sch")
 		(attr through_hole)
 		(duplicate_pad_numbers_are_jumpers no)
@@
 		(property ki_fp_filters "Connector*:*_2x??_*")
 		(sheetname "/")
-		(sheetfile "Dev Board.kicad_sch")
+		(sheetfile "DEV Board.kicad_sch")
 		(attr through_hole)
 		(duplicate_pad_numbers_are_jumpers no)
@@
 		(property ki_fp_filters "Connector*:*_1x??_*")
 		(sheetname "/")
-		(sheetfile "Dev Board.kicad_sch")
+		(sheetfile "DEV Board.kicad_sch")
 		(units
 			(unit
@@
 		(property ki_fp_filters "R_*")
 		(sheetname "/")
-		(sheetfile "Dev Board.kicad_sch")
+		(sheetfile "DEV Board.kicad_sch")
 		(units
 			(unit
@@
 		)
 		(sheetname "/")
-		(sheetfile "Dev Board.kicad_sch")
+		(sheetfile "DEV Board.kicad_sch")
 		(units
 			(unit
@@
 		)
 		(sheetname "/")
-		(sheetfile "Dev Board.kicad_sch")
+		(sheetfile "DEV Board.kicad_sch")
 		(units
 			(unit
@@
 		(property ki_fp_filters "Connector*:*_2x??_*")
 		(sheetname "/")
-		(sheetfile "Dev Board.kicad_sch")
+		(sheetfile "DEV Board.kicad_sch")
 		(units
 			(unit
@@
 		(property ki_fp_filters "C_*")
 		(sheetname "/")
-		(sheetfile "Dev Board.kicad_sch")
+		(sheetfile "DEV Board.kicad_sch")
 		(units
 			(unit
@@
 		(property ki_fp_filters "C_*")
 		(sheetname "/")
-		(sheetfile "Dev Board.kicad_sch")
+		(sheetfile "DEV Board.kicad_sch")
 		(units
 			(unit
@@
 		(property ki_fp_filters "R_*")
 		(sheetname "/")
-		(sheetfile "Dev Board.kicad_sch")
+		(sheetfile "DEV Board.kicad_sch")
 		(units
 			(unit
@@
 		(property ki_fp_filters "R_*")
 		(sheetname "/")
-		(sheetfile "Dev Board.kicad_sch")
+		(sheetfile "DEV Board.kicad_sch")
 		(units
 			(unit
@@
 		(property ki_fp_filters "USB*C*Receptacle*")
 		(sheetname "/")
-		(sheetfile "Dev Board.kicad_sch")
+		(sheetfile "DEV Board.kicad_sch")
 		(attr smd)
 		(duplicate_pad_numbers_are_jumpers no)
@@
 		(property ki_fp_filters "C_*")
 		(sheetname "/")
-		(sheetfile "Dev Board.kicad_sch")
+		(sheetfile "DEV Board.kicad_sch")
 		(units
 			(unit
@@
 		(property ki_fp_filters "C_*")
 		(sheetname "/")
-		(sheetfile "Dev Board.kicad_sch")
+		(sheetfile "DEV Board.kicad_sch")
 		(units
 			(unit
@@
 		(property ki_fp_filters "R_*")
 		(sheetname "/")
-		(sheetfile "Dev Board.kicad_sch")
+		(sheetfile "DEV Board.kicad_sch")
 		(units
 			(unit
@@
 		)
 		(sheetname "/")
-		(sheetfile "Dev Board.kicad_sch")
+		(sheetfile "DEV Board.kicad_sch")
 		(attr through_hole)
 		(duplicate_pad_numbers_are_jumpers no)
@@
 		(property ki_fp_filters "8P8C* RJ45*")
 		(sheetname "/")
-		(sheetfile "Dev Board.kicad_sch")
+		(sheetfile "DEV Board.kicad_sch")
 		(attr through_hole)
 		(duplicate_pad_numbers_are_jumpers no)
@@
 		)
 		(sheetname "/")
-		(sheetfile "Dev Board.kicad_sch")
+		(sheetfile "DEV Board.kicad_sch")
 		(units
 			(unit
@@
 		(property ki_fp_filters "C_*")
 		(sheetname "/")
-		(sheetfile "Dev Board.kicad_sch")
+		(sheetfile "DEV Board.kicad_sch")
 		(units
 			(unit
@@
 		(property ki_fp_filters "R_*")
 		(sheetname "/")
-		(sheetfile "Dev Board.kicad_sch")
+		(sheetfile "DEV Board.kicad_sch")
 		(units
 			(unit
@@
 		(property ki_fp_filters "R_*")
 		(sheetname "/")
-		(sheetfile "Dev Board.kicad_sch")
+		(sheetfile "DEV Board.kicad_sch")
 		(units
 			(unit
@@
 		(property ki_fp_filters "C_*")
 		(sheetname "/")
-		(sheetfile "Dev Board.kicad_sch")
+		(sheetfile "DEV Board.kicad_sch")
 		(units
 			(unit
@@
 		)
 		(sheetname "/")
-		(sheetfile "Dev Board.kicad_sch")
+		(sheetfile "DEV Board.kicad_sch")
 		(units
 			(unit
