File: Hardware/Dev Board/Rev 1.0/Dev Board.kicad_sch (KiCad schematic)
At the start: 39 parts, among them J1 VBAT, J2 SPI, J3 PANEL, J4 6502 Card Connector, J5 6502 Bus, J6 USB Host, J7 USB HOST, J8 RJ45_LED, J9 ETHERNET, SW1 Run/Stop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

Commit message: Cleanup DEV project
Connections:
- net GND: now also J6.SH (SHIELD); no longer J6.S1 (SHIELD)

Commit message: Uppercase DEV
Other:
- title: 6502 Dev Board -> 6502 DEV Board
Changed lines of the file:
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@@
 	(paper "USLedger")
 	(title_block
-		(title "6502 Dev Board")
+		(title "6502 DEV Board")
 		(date "2025-09-26")
 		(rev "1.0")
@@
 		)
 		(instances
-			(project "Dev Board"
+			(project "DEV Board"
 				(path "/5d95bc66-f610-41ca-b1ae-73f5b5edc5a7"
 					(reference "J5")
@@
 		)
 		(instances
-			(project "Dev Board"
+			(project "DEV Board"
 				(path "/5d95bc66-f610-41ca-b1ae-73f5b5edc5a7"
 					(reference "C6")
@@
 		)
 		(instances
-			(project "Dev Board"
+			(project "DEV Board"
 				(path "/5d95bc66-f610-41ca-b1ae-73f5b5edc5a7"
 					(reference "C7")
@@
 		)
 		(instances
-			(project "Dev Board"
+			(project "DEV Board"
 				(path "/5d95bc66-f610-41ca-b1ae-73f5b5edc5a7"
 					(reference "U4")
@@
 		)
 		(instances
-			(project "Dev Board"
+			(project "DEV Board"
 				(path "/5d95bc66-f610-41ca-b1ae-73f5b5edc5a7"
 					(reference "C8")
@@
 		)
 		(instances
-			(project "Dev Board"
+			(project "DEV Board"
 				(path "/5d95bc66-f610-41ca-b1ae-73f5b5edc5a7"
 					(reference "R9")
@@
 		)
 		(instances
-			(project "Dev Board"
+			(project "DEV Board"
 				(path "/5d95bc66-f610-41ca-b1ae-73f5b5edc5a7"
 					(reference "R4")
@@
 		)
 		(instances
-			(project "Dev Board"
+			(project "DEV Board"
 				(path "/5d95bc66-f610-41ca-b1ae-73f5b5edc5a7"
 					(reference "U5")
@@
 		)
 		(instances
-			(project "Dev Board"
+			(project "DEV Board"
 				(path "/5d95bc66-f610-41ca-b1ae-73f5b5edc5a7"
 					(reference "J9")
@@
 		)
 		(instances
-			(project "Dev Board"
+			(project "DEV Board"
 				(path "/5d95bc66-f610-41ca-b1ae-73f5b5edc5a7"
 					(reference "C1")
@@
 		)
 		(instances
-			(project "Dev Board"
+			(project "DEV Board"
 				(path "/5d95bc66-f610-41ca-b1ae-73f5b5edc5a7"
 					(reference "#PWR07")
@@
 		)
 		(instances
-			(project "Dev Board"
+			(project "DEV Board"
 				(path "/5d95bc66-f610-41ca-b1ae-73f5b5edc5a7"
 					(reference "R8")
@@
 		)
 		(instances
-			(project "Dev Board"
+			(project "DEV Board"
 				(path "/5d95bc66-f610-41ca-b1ae-73f5b5edc5a7"
 					(reference "J2")
@@
 		)
 		(instances
-			(project "Dev Board"
+			(project "DEV Board"
 				(path "/5d95bc66-f610-41ca-b1ae-73f5b5edc5a7"
 					(reference "J8")
@@
 		)
 		(instances
-			(project "Dev Board"
+			(project "DEV Board"
 				(path "/5d95bc66-f610-41ca-b1ae-73f5b5edc5a7"
 					(reference "U1")
@@
 		)
 		(instances
-			(project "Dev Board"
+			(project "DEV Board"
 				(path "/5d95bc66-f610-41ca-b1ae-73f5b5edc5a7"
 					(reference "J7")
@@
 		)
 		(instances
-			(project "Dev Board"
+			(project "DEV Board"
 				(path "/5d95bc66-f610-41ca-b1ae-73f5b5edc5a7"
 					(reference "#PWR013")
@@
 		)
 		(instances
-			(project "Dev Board"
+			(project "DEV Board"
 				(path "/5d95bc66-f610-41ca-b1ae-73f5b5edc5a7"
 					(reference "#FLG02")
@@
 		)
 		(instances
-			(project "Dev Board"
+			(project "DEV Board"
 				(path "/5d95bc66-f610-41ca-b1ae-73f5b5edc5a7"
 					(reference "#PWR011")
@@
 		)
 		(instances
-			(project "Dev Board"
+			(project "DEV Board"
 				(path "/5d95bc66-f610-41ca-b1ae-73f5b5edc5a7"
 					(reference "SW3")
@@
 		)
 		(instances
-			(project "Dev Board"
+			(project "DEV Board"
 				(path "/5d95bc66-f610-41ca-b1ae-73f5b5edc5a7"
 					(reference "#PWR02")
@@
 		)
 		(instances
-			(project "Dev Board"
+			(project "DEV Board"
 				(path "/5d95bc66-f610-41ca-b1ae-73f5b5edc5a7"
 					(reference "#FLG03")
@@
 		)
 		(instances
-			(project "Dev Board"
+			(project "DEV Board"
 				(path "/5d95bc66-f610-41ca-b1ae-73f5b5edc5a7"
 					(reference "SW4")
@@
 		)
 		(instances
-			(project "Dev Board"
+			(project "DEV Board"
 				(path "/5d95bc66-f610-41ca-b1ae-73f5b5edc5a7"
 					(reference "J3")
@@
 		)
 		(instances
-			(project "Dev Board"
+			(project "DEV Board"
 				(path "/5d95bc66-f610-41ca-b1ae-73f5b5edc5a7"
 					(reference "J1")
@@
 		)
 		(instances
-			(project "Dev Board"
+			(project "DEV Board"
 				(path "/5d95bc66-f610-41ca-b1ae-73f5b5edc5a7"
 					(reference "R6")
@@
 		)
 		(instances
-			(project "Dev Board"
+			(project "DEV Board"
 				(path "/5d95bc66-f610-41ca-b1ae-73f5b5edc5a7"
 					(reference "#PWR01")
@@
 		)
 		(instances
-			(project "Dev Board"
+			(project "DEV Board"
 				(path "/5d95bc66-f610-41ca-b1ae-73f5b5edc5a7"
 					(reference "R3")
@@
 		)
 		(instances
-			(project "Dev Board"
+			(project "DEV Board"
 				(path "/5d95bc66-f610-41ca-b1ae-73f5b5edc5a7"
 					(reference "#PWR04")
@@
 		)
 		(instances
-			(project "Dev Board"
+			(project "DEV Board"
 				(path "/5d95bc66-f610-41ca-b1ae-73f5b5edc5a7"
 					(reference "R11")
@@
 		)
 		(instances
-			(project "Dev Board"
+			(project "DEV Board"
 				(path "/5d95bc66-f610-41ca-b1ae-73f5b5edc5a7"
 					(reference "#PWR012")
@@
 		)
 		(instances
-			(project "Dev Board"
+			(project "DEV Board"
 				(path "/5d95bc66-f610-41ca-b1ae-73f5b5edc5a7"
 					(reference "R2")
@@
 		)
 		(instances
-			(project "Dev Board"
+			(project "DEV Board"
 				(path "/5d95bc66-f610-41ca-b1ae-73f5b5edc5a7"
 					(reference "#PWR08")
@@
 		)
 		(instances
-			(project "Dev Board"
+			(project "DEV Board"
 				(path "/5d95bc66-f610-41ca-b1ae-73f5b5edc5a7"
 					(reference "SW2")
@@
 		)
 		(instances
-			(project "Dev Board"
+			(project "DEV Board"
 				(path "/5d95bc66-f610-41ca-b1ae-73f5b5edc5a7"
 					(reference "#PWR06")
@@
 		)
 		(instances
-			(project "Dev Board"
+			(project "DEV Board"
 				(path "/5d95bc66-f610-41ca-b1ae-73f5b5edc5a7"
 					(reference "#PWR018")
@@
 		)
 		(instances
-			(project "Dev Board"
+			(project "DEV Board"
 				(path "/5d95bc66-f610-41ca-b1ae-73f5b5edc5a7"
 					(reference "SW1")
@@
 		)
 		(instances
-			(project "Dev Board"
+			(project "DEV Board"
 				(path "/5d95bc66-f610-41ca-b1ae-73f5b5edc5a7"
 					(reference "#FLG04")
@@
 		)
 		(instances
-			(project "Dev Board"
+			(project "DEV Board"
 				(path "/5d95bc66-f610-41ca-b1ae-73f5b5edc5a7"
 					(reference "R5")
@@
 		)
 		(instances
-			(project "Dev Board"
+			(project "DEV Board"
 				(path "/5d95bc66-f610-41ca-b1ae-73f5b5edc5a7"
 					(reference "R10")
@@
 		)
 		(instances
-			(project "Dev Board"
+			(project "DEV Board"
 				(path "/5d95bc66-f610-41ca-b1ae-73f5b5edc5a7"
 					(reference "R7")
@@
 		)
 		(instances
-			(project "Dev Board"
+			(project "DEV Board"
 				(path "/5d95bc66-f610-41ca-b1ae-73f5b5edc5a7"
 					(reference "C5")
@@
 		)
 		(instances
-			(project "Dev Board"
+			(project "DEV Board"
 				(path "/5d95bc66-f610-41ca-b1ae-73f5b5edc5a7"
 					(reference "U2")
@@
 		)
 		(instances
-			(project "Dev Board"
+			(project "DEV Board"
 				(path "/5d95bc66-f610-41ca-b1ae-73f5b5edc5a7"
 					(reference "#PWR010")
@@
 		)
 		(instances
-			(project "Dev Board"
+			(project "DEV Board"
 				(path "/5d95bc66-f610-41ca-b1ae-73f5b5edc5a7"
 					(reference "#PWR016")
@@
 		)
 		(instances
-			(project "Dev Board"
+			(project "DEV Board"
 				(path "/5d95bc66-f610-41ca-b1ae-73f5b5edc5a7"
 					(reference "U6")
@@
 		)
 		(instances
-			(project "Dev Board"
+			(project "DEV Board"
 				(path "/5d95bc66-f610-41ca-b1ae-73f5b5edc5a7"
 					(reference "#PWR03")
@@
 		)
 		(instances
-			(project "Dev Board"
+			(project "DEV Board"
 				(path "/5d95bc66-f610-41ca-b1ae-73f5b5edc5a7"
 					(reference "#PWR017")
@@
 		)
 		(instances
-			(project "Dev Board"
+			(project "DEV Board"
 				(path "/5d95bc66-f610-41ca-b1ae-73f5b5edc5a7"
 					(reference "#FLG01")
@@
 		)
 		(instances
-			(project "Dev Board"
+			(project "DEV Board"
 				(path "/5d95bc66-f610-41ca-b1ae-73f5b5edc5a7"
 					(reference "C3")
@@
 		)
 		(instances
-			(project "Dev Board"
+			(project "DEV Board"
 				(path "/5d95bc66-f610-41ca-b1ae-73f5b5edc5a7"
 					(reference "R1")
@@
 		)
 		(instances
-			(project "Dev Board"
+			(project "DEV Board"
 				(path "/5d95bc66-f610-41ca-b1ae-73f5b5edc5a7"
 					(reference "C4")
@@
 		)
 		(instances
-			(project "Dev Board"
+			(project "DEV Board"
 				(path "/5d95bc66-f610-41ca-b1ae-73f5b5edc5a7"
 					(reference "J4")
@@
 		)
 		(instances
-			(project "Dev Board"
+			(project "DEV Board"
 				(path "/5d95bc66-f610-41ca-b1ae-73f5b5edc5a7"
 					(reference "#PWR014")
@@
 		)
 		(instances
-			(project "Dev Board"
+			(project "DEV Board"
 				(path "/5d95bc66-f610-41ca-b1ae-73f5b5edc5a7"
 					(reference "#PWR09")
@@
 		)
 		(instances
-			(project "Dev Board"
+			(project "DEV Board"
 				(path "/5d95bc66-f610-41ca-b1ae-73f5b5edc5a7"
 					(reference "C2")
@@
 		)
 		(instances
-			(project "Dev Board"
+			(project "DEV Board"
 				(path "/5d95bc66-f610-41ca-b1ae-73f5b5edc5a7"
 					(reference "BT1")
@@
 		)
 		(instances
-			(project "Dev Board"
+			(project "DEV Board"
 				(path "/5d95bc66-f610-41ca-b1ae-73f5b5edc5a7"
 					(reference "U3")
@@
 		)
 		(instances
-			(project "Dev Board"
+			(project "DEV Board"
 				(path "/5d95bc66-f610-41ca-b1ae-73f5b5edc5a7"
 					(reference "#PWR015")
@@
 		)
 		(instances
-			(project "Dev Board"
+			(project "DEV Board"
 				(path "/5d95bc66-f610-41ca-b1ae-73f5b5edc5a7"
 					(reference "#PWR05")
@@
 		)
 		(instances
-			(project "Dev Board"
+			(project "DEV Board"
 				(path "/5d95bc66-f610-41ca-b1ae-73f5b5edc5a7"
 					(reference "J6")
