File: Hardware/Dev Output Board/Rev 1.0/Dev Output Board.kicad_pcb (KiCad board)
At the start: 2 copper layers, 100 x 100 mm, 14 parts, among them J1 SPEAKER, J2 SERIAL, U1 Waveshare 2.4in LCD Header, U2 Teensy4.0, U3 Waveshare 2.4in LCD

Commit message: Uppercase DEV
Parts:
- G***: footprint 6502 Logos:6502 Dev Output Board Logo 4mm -> 6502 Logos:6502 DEV Output Board Logo 4mm
Changed lines of the file:
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@@
 	(paper "USLetter")
 	(title_block
-		(title "6502 Dev Output Board")
+		(title "6502 DEV Output Board")
 		(date "2025-12-06")
 		(rev "1.0")
@@
 		(property ki_fp_filters "MountingHole*")
 		(sheetname "/")
-		(sheetfile "Dev Board.kicad_sch")
+		(sheetfile "DEV Board.kicad_sch")
 		(attr board_only exclude_from_pos_files exclude_from_bom)
 		(duplicate_pad_numbers_are_jumpers no)
@@
 		(property ki_fp_filters "MountingHole*")
 		(sheetname "/")
-		(sheetfile "Dev Board.kicad_sch")
+		(sheetfile "DEV Board.kicad_sch")
 		(attr board_only exclude_from_pos_files exclude_from_bom)
 		(duplicate_pad_numbers_are_jumpers no)
@@
 		(property ki_fp_filters "MountingHole*")
 		(sheetname "/")
-		(sheetfile "Dev Board.kicad_sch")
+		(sheetfile "DEV Board.kicad_sch")
 		(attr board_only exclude_from_pos_files exclude_from_bom)
 		(duplicate_pad_numbers_are_jumpers no)
@@
 		(property ki_fp_filters "MountingHole*")
 		(sheetname "/")
-		(sheetfile "Dev Board.kicad_sch")
+		(sheetfile "DEV Board.kicad_sch")
 		(attr board_only exclude_from_pos_files exclude_from_bom)
 		(duplicate_pad_numbers_are_jumpers no)
@@
 		(property ki_fp_filters "C_*")
 		(sheetname "/")
-		(sheetfile "Dev Output Board.kicad_sch")
+		(sheetfile "DEV Output Board.kicad_sch")
 		(attr through_hole)
 		(duplicate_pad_numbers_are_jumpers no)
@@
 		(embedded_fonts no)
 	)
-	(footprint "6502 Logos:6502 Dev Output Board Logo 4mm"
+	(footprint "6502 Logos:6502 DEV Output Board Logo 4mm"
 		(layer "F.Cu")
 		(at 161.888339 56.049876 180)
@@
 		)
 		(sheetname "/")
-		(sheetfile "Dev Output Board.kicad_sch")
+		(sheetfile "DEV Output Board.kicad_sch")
 		(attr through_hole)
 		(duplicate_pad_numbers_are_jumpers no)
@@
 		(property ki_fp_filters "R_*")
 		(sheetname "/")
-		(sheetfile "Dev Output Board.kicad_sch")
+		(sheetfile "DEV Output Board.kicad_sch")
 		(attr through_hole)
 		(duplicate_pad_numbers_are_jumpers no)
@@
 		)
 		(sheetname "/")
-		(sheetfile "Dev Output Board.kicad_sch")
+		(sheetfile "DEV Output Board.kicad_sch")
 		(attr through_hole exclude_from_bom)
 		(duplicate_pad_numbers_are_jumpers no)
@@
 		)
 		(sheetname "/")
-		(sheetfile "Dev Output Board.kicad_sch")
+		(sheetfile "DEV Output Board.kicad_sch")
 		(attr through_hole)
 		(duplicate_pad_numbers_are_jumpers no)
@@
 		(property ki_fp_filters "Connector*:*_1x??_*")
 		(sheetname "/")
-		(sheetfile "Dev Output Board.kicad_sch")
+		(sheetfile "DEV Output Board.kicad_sch")
 		(attr through_hole)
 		(duplicate_pad_numbers_are_jumpers no)
@@
 		(property ki_fp_filters "Connector*:*_1x??_*")
 		(sheetname "/")
-		(sheetfile "Dev Output Board.kicad_sch")
+		(sheetfile "DEV Output Board.kicad_sch")
 		(attr through_hole)
 		(duplicate_pad_numbers_are_jumpers no)
