File: Hardware/Dev Output Board/Rev 1.0/Dev Output Board.kicad_sch (KiCad schematic)
At the start: 7 parts, among them J1 SPEAKER, J2 SERIAL, U1 Waveshare 2.4in LCD Header, U2 Teensy4.0, U3 Waveshare 2.4in LCD

Commit message: Uppercase DEV
Other:
- title: 6502 Dev Output Board -> 6502 DEV Output Board
Changed lines of the file:
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@@
 	(paper "USLetter")
 	(title_block
-		(title "6502 Dev Output Board")
+		(title "6502 DEV Output Board")
 		(date "2025-12-06")
 		(rev "1.0")
@@
 		)
 		(instances
-			(project "Dev Output Board"
+			(project "DEV Output Board"
 				(path "/5d95bc66-f610-41ca-b1ae-73f5b5edc5a7"
 					(reference "J1")
@@
 		)
 		(instances
-			(project "Dev Output Board"
+			(project "DEV Output Board"
 				(path "/5d95bc66-f610-41ca-b1ae-73f5b5edc5a7"
 					(reference "U1")
@@
 		)
 		(instances
-			(project "Dev Output Board"
+			(project "DEV Output Board"
 				(path "/5d95bc66-f610-41ca-b1ae-73f5b5edc5a7"
 					(reference "J2")
@@
 		)
 		(instances
-			(project "Dev Output Board"
+			(project "DEV Output Board"
 				(path "/5d95bc66-f610-41ca-b1ae-73f5b5edc5a7"
 					(reference "#PWR04")
@@
 		)
 		(instances
-			(project "Dev Output Board"
+			(project "DEV Output Board"
 				(path "/5d95bc66-f610-41ca-b1ae-73f5b5edc5a7"
 					(reference "C1")
@@
 		)
 		(instances
-			(project "Dev Output Board"
+			(project "DEV Output Board"
 				(path "/5d95bc66-f610-41ca-b1ae-73f5b5edc5a7"
 					(reference "R6")
@@
 		)
 		(instances
-			(project "Dev Output Board"
+			(project "DEV Output Board"
 				(path "/5d95bc66-f610-41ca-b1ae-73f5b5edc5a7"
 					(reference "#PWR010")
@@
 		)
 		(instances
-			(project "Dev Output Board"
+			(project "DEV Output Board"
 				(path "/5d95bc66-f610-41ca-b1ae-73f5b5edc5a7"
 					(reference "U2")
@@
 		)
 		(instances
-			(project "Dev Output Board"
+			(project "DEV Output Board"
 				(path "/5d95bc66-f610-41ca-b1ae-73f5b5edc5a7"
 					(reference "#PWR03")
@@
 		)
 		(instances
-			(project "Dev Output Board"
+			(project "DEV Output Board"
 				(path "/5d95bc66-f610-41ca-b1ae-73f5b5edc5a7"
 					(reference "#PWR06")
@@
 		)
 		(instances
-			(project "Dev Output Board"
+			(project "DEV Output Board"
 				(path "/5d95bc66-f610-41ca-b1ae-73f5b5edc5a7"
 					(reference "U3")
@@
 		)
 		(instances
-			(project "Dev Output Board"
+			(project "DEV Output Board"
 				(path "/5d95bc66-f610-41ca-b1ae-73f5b5edc5a7"
 					(reference "#PWR02")
